Commit message: provide a working functional attitude controller and copter

File: rrbot_description/urdf/rrbot.xacro (robot description, xacro)
@@ -318,8 +318,20 @@
     <xacro:motor_with_propeller_right name="motor0" />
     <joint name="bar_motor1_joint" type="fixed">
+        <parent link="bar0"/>
+        <origin xyz="0.18 0 0.02" rpy="0 0 0"/>
+        <child link="motor1_link"/>
+    </joint>
+    <xacro:motor_with_propeller_left name="motor1" />
+    <joint name="bar_motor2_joint" type="fixed">
         <parent link="bar1"/>
         <origin xyz="-0.18 0 0.02" rpy="0 0 0"/>
-        <child link="motor1_link"/>
-    </joint>
-    <xacro:motor_with_propeller_left name="motor1" />
+        <child link="motor2_link"/>
+    </joint>
+    <xacro:motor_with_propeller_right name="motor2" />
+    <joint name="bar_motor3_joint" type="fixed">
+        <parent link="bar0"/>
+        <origin xyz="-0.18 0 0.02" rpy="0 0 0"/>
+        <child link="motor3_link"/>
+    </joint>
+    <xacro:motor_with_propeller_left name="motor3" />
 </robot>

Commit message: control modification -- convert to NED before applying control

File: rrbot_description/urdf/rrbot.xacro (robot description, xacro)
@@ -215,5 +215,5 @@
             <actuator name="${name}">
                 <hardwareInterface>hardware_interface/EffortJointInterface</hardwareInterface>
-                <mechanicalReduction>1</mechanicalReduction>
+                <mechanicalReduction>0</mechanicalReduction>
             </actuator>
             </transmission>
@@ -288,5 +288,5 @@
     <joint name="FC_joint" type="fixed">
         <parent link="dummyroot"/>
-        <origin xyz="0 0 0.01" rpy="0 0 0"/>
+	<origin xyz="0 0 0.01" rpy="0 0 0"/>
         <child link="FC"/>
     </joint>
